File: X-B120W-4-LITE-120W-CLASS-B-POWER-AMP-SIMPLE-MAIN-CIRCUIT.kicad_pcb (KiCad board)
At the start: 2 copper layers, 149.2 x 66.7 mm, 83 parts, among them Q4001 2N5401, Q4002 2N5401, Q4003 2N5401, Q4004 2N5551, Q4005 2N5551, Q4006 2N5551, Q4007 2N5551, Q4008 2N5551, Q4009 2N5401, Q4010 2N5551, Q4011 TIP41A, Q4012 TIP42C, Q4013 2SC5200, Q4014 2SA1943

Commit message: Update
Other:
- board text added: "X-B120W-4-LITE"
Changed lines of the file:
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@@
+		)
+	)
+	(gr_text "X-B120W-4-LITE"
+		(at 66.675 148.59 90)
+		(layer "F.SilkS")
+		(effects
+			(font
+				(size 2 2)
+				(thickness 0.15)
+			)
 		)
 	)
@@
 		)
 	)
+	(gr_text "X-B120W-4-LITE"
+		(at 210.185 148.7875 90)
+		(layer "B.SilkS")
+		(effects
+			(font
+				(size 2 2)
+				(thickness 0.15)
+			)
+			(justify mirror)
+		)
+	)
