File: X-B120W-4-LITE-120W-CLASS-B-POWER-AMP-SIMPLE-MAIN-CIRCUIT.kicad_sch (KiCad schematic)
At the start: 87 parts, among them Q4001 2N5401, Q4002 2N5401, Q4003 2N5401, Q4004 2N5551, Q4005 2N5551, Q4006 2N5551, Q4007 2N5551, Q4008 2N5551, Q4009 2N5401, Q4010 2N5551, Q4011 TIP41A, Q4012 TIP42C, Q4013 2SC5200, Q4014 2SA1943

Commit message: Update
Other:
- note added: ".PARAM R_LOAD=4"
- note removed: ".PARAM R_LOAD=1"
Changed lines of the file:
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@@
 		)
 	)
-	(text ".PARAM R_LOAD=1"
+	(text ".PARAM R_LOAD=4"
 		(exclude_from_sim no)
 		(at -62.23 67.31 0)
